File: HW/eagle/daGloane.brd (EAGLE design)
At the start: 182.4 x 160.7 mm, 110 parts, among them IC1 MCP1252-33X50, U1 STM32F10XTXU6, X2 SPARKFUN-CONNECTORS_USB-MICROB

Commit message: led added to LiPo charge IC
Parts:
- added LED5: (no value), led:CHIPLED_0805
- added R29: 330, rcl:R0603
Connections:
- new net N$43: R29.2, U$2.1
- new net N$44: LED5.C, R29.1
- net VBUS: now also LED5.A; no longer U$2.1
Changed lines of the file:
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@@
 <element name="R28" library="rcl" package="R0603" value="10k" x="1.5" y="-151.2"/>
 <element name="D5" library="diode" package="SOD123" value="MBR0520LT" x="2.7" y="-145.8"/>
+<element name="LED5" library="led" package="CHIPLED_0805" value="" x="-3.1" y="-162.5"/>
+<element name="R29" library="rcl" package="R0603" value="330" x="-4.5" y="-167"/>
 </elements>
 <signals>
@@
 <contactref element="U$4" pad="10"/>
 <contactref element="C16" pad="1"/>
-<contactref element="U$2" pad="1"/>
 <contactref element="U$2" pad="4"/>
 <contactref element="C6" pad="2"/>
 <contactref element="X2" pad="VBUS"/>
-<wire x1="56.45" y1="39.2" x2="54.45" y2="47.675" width="0" layer="19" extent="1-1"/>
-<wire x1="53.5" y1="37.75" x2="56.45" y2="39.2" width="0" layer="19" extent="1-1"/>
-<wire x1="48.5" y1="29.85" x2="53.5" y2="37.75" width="0" layer="19" extent="1-1"/>
-<wire x1="46.95" y1="29.8001" x2="48.5" y2="29.85" width="0" layer="19" extent="1-1"/>
-<wire x1="45.05" y1="27.1999" x2="46.95" y2="29.8001" width="0" layer="19" extent="1-1"/>
+<contactref element="LED5" pad="A"/>
+<wire x1="45.05" y1="27.1999" x2="-3.1" y2="-163.55" width="0" layer="19" extent="1-1"/>
+<wire x1="48.5" y1="29.85" x2="45.05" y2="27.1999" width="0" layer="19" extent="1-1"/>
+<wire x1="53.5" y1="37.75" x2="48.5" y2="29.85" width="0" layer="19" extent="1-1"/>
+<wire x1="56.45" y1="39.2" x2="53.5" y2="37.75" width="0" layer="19" extent="1-1"/>
+<wire x1="54.45" y1="47.675" x2="56.45" y2="39.2" width="0" layer="19" extent="1-1"/>
 </signal>
 <signal name="N$5">
@@
 <wire x1="4.6" y1="-145.8" x2="1.3" y2="-160.3" width="0" layer="19" extent="1-1"/>
 </signal>
+<signal name="N$43">
+<contactref element="U$2" pad="1"/>
+<contactref element="R29" pad="2"/>
+<wire x1="46.95" y1="29.8001" x2="-3.65" y2="-167" width="0" layer="19" extent="1-1"/>
+</signal>
+<signal name="N$44">
+<contactref element="R29" pad="1"/>
+<contactref element="LED5" pad="C"/>
+<wire x1="-3.1" y1="-161.45" x2="-5.35" y2="-167" width="0" layer="19" extent="1-1"/>
+</signal>
 </signals>

Commit message: - PI filter added to charge pump DC/DC - trough hole pads for BLDC motors replaced with SMT type pads
Parts:
- added C30, C31: 10µF/6.3V, rcl:C0805
- added L1, L2: (no value), daGloane:WUERTH-ELEKTRONIK_WE-KI_0805_B
- MOT1_A, MOT1_B, MOT1_C, MOT2_A, MOT2_B, MOT2_C, MOT3_A, MOT3_B, MOT3_C, MOT4_A, MOT4_B, MOT4_C: value WIREPAD1,6/0,8 -> WIREPADSMD1,27-254; device wirepad:1,6/0,8 -> wirepad:SMD1,27-2,54
- moved MOT1_C 9.17 mm to (9.60, 11.0), turned to 315 degrees
- moved C23 9.11 mm to (24.3, 15.6), turned to 135 degrees
- moved C22 3.84 mm to (26.2, 13.4), turned to 225 degrees
- moved U$6 3.22 mm to (21.4, 10.6), turned to 315 degrees
- moved MOT1_A 1.39 mm to (10.9, 9.62), turned to 315 degrees
- moved MOT1_B 1.25 mm to (12.6, 8.05), turned to 315 degrees
Connections:
- new net N$45: C12.1, IC1.3, L2.1
- new net N$46: C13.1, IC1.2, L1.2
- net GND: now also C30.2, C31.2
- net LIPO: now also C30.1, L2.2; no longer C12.1, IC1.3
- net VCC: now also C31.1, L1.1; no longer C13.1, IC1.2

Commit message: 100nF capacitor added to PI filters of charge pump dc/dc series resistors of spi resized to 150R
Parts:
- removed R18: 3k3, rcl:R0603
- added C32, C33: 100nF, rcl:C0603
- LED1, LED2, LED3, LED4, LED5: device led:CHIPLED_0805 -> led:CHIPLED_0603
- R1, R3, R4, R5: value 1k -> 150R
- R17: value 3k3 -> 10k
Connections:
- removed net N$22: C20.1, R12.1, R18.2, R21.2
- net GND: now also C32.1, C33.1
- net LIPO: now also C32.2
- net VCC: now also C33.2
- net VOLTAGE: now also C20.1, R12.1, R21.2; no longer R18.1
